File: LED_breakout_top.sch (KiCad schematic (older format))
At the start: 24 parts, among them P1 CONN_5, P10 CONN_2, P11 CONN_2, P13 CONN_2, P14 CONN_2, P16 CONN_2, P17 CONN_2, P2 CONN_5, P20 CONN_1, P21 CONN_1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

Commit message: Update LED_breakout_top
Updated to use the new Joes_Discrete lib so that an easy BOM can be created
Parts:
- removed C101, C102, C103, C104: C, symbol C
- removed D10: ZENER, symbol ZENER
- removed P1, P2: CONN_5, symbol CONN_5
- removed P10, P11, P13, P14, P16, P17: CONN_2, symbol CONN_2
- removed Q10: SI2308BDS, symbol MOSFET_N
- removed R10: 100K, symbol R
- removed R102, R103, R11: 0-ohm, symbol R
- added C101, C102: CAP_2P2UF_10P_50V_X5R_1206, symbol CAP_2P2UF_10P_50V_X5R_1206
- added C103, C104: CAP_0P1UF_10P_50V_X7R_0805, symbol CAP_0P1UF_10P_50V_X7R_0805
- added D10: DIODE_ZENER_9P1V, symbol DIODE_ZENER_9P1V
- added P1, P2: CONN_TE_CT_5, symbol CONN_TE_CT_5
- added P10, P11, P13, P14, P16, P17: CONN_JST_PH_2, symbol CONN_JST_PH_2
- added Q10: MOS_N_SI2308BDS, symbol MOS_N_SI2308BDS
- added R10: RES_100K_1P_1V8W_0805, symbol RES_100K_1P_1V8W_0805
- added R102, R103, R11: RES_0_0P_1V4_1206, symbol RES_0_0P_1V4_1206
Connections:
- wire segments 41 -> 40
