File: New_Kitchen_LM3414.sch (KiCad schematic (older format))
At the start: 109 parts, among them IC101 LPC1343, J101 USB_MINI_B, J102 USB_MINI_B, K101 CONN_3, P101 CONN_2, P102 CONN_2, P103 CONN_5X2, P104 CONN_2, P105 CONN_2, P106 CONN_5, Q101 MOSFET_N, Q102 MOSFET_P, SW101 SW_PUSH, SW102 SW_PUSH, U101 VREG_1117, U102 XBEE, U103 FT232RL, U150 LM3414, U160 LM3414, U170 LM3414, U180 LM3414, U190 LM3414, X101 CRYSTAL

Commit message: layout is preliminary finalize.  I still need to develop a devel board.  It will have all the same functionality without all the wires and stuff.  Just LEDs for each function
Parts:
- added C1, C14, C15, C16, C2, C4, C8, C9: C, symbol C
- added C11, C12, C13, C3, C5, C6: CP1, symbol CP1
- added D1, D2: DIODE, symbol DIODE
- added HW100, HW101, HW102, HW103: CONN_1, symbol CONN_1
- added K1: CONN_3, symbol CONN_3
- added P1: CONN_4, symbol CONN_4
- added R1, R2: R, symbol R
- C103: PN (none) -> 1234
Connections:
- net +24V: now also C11.1, C12.1, C13.1, C14.1, C15.1, C16.1, C3.1, C4.1, C5.1, C6.1, C8.1, C9.1
- net +3.3V: now also P103.1, C1.1, K1.1 (P1), P1.1 (P1), R1.1, R2.1; no longer P103.9
- net AD1: now also P103.10; no longer P103.2
- net AD2: now also P103.9; no longer P103.1
- net AD3: now also P103.8; no longer P103.4
- net AD4: now also P103.7; no longer P103.3
- net BLU_DIM: now also IC101.40 (PIO1_4-AD5-CT32B1_MAT3-WAKEUP); no longer IC101.27 (PIO0_8-MISO-CT16B0_MAT0)
- net BOOT_SEL: now also C123.1, D108.1 (A), R110.2, D1.1 (A), D2.1 (A); no longer U102.16 (/RTS/AD6/Dio6), U103.3 (RTS)
- net GND: now also P103.3, C1.2, C11.2, C12.2, C13.2, C14.2, C15.2, C16.2, C2.2, C3.2, C4.2, C5.2, C6.2, C8.2, C9.2, K1.3 (P3), P1.4 (P4); no longer P103.7
- net GRN_DIM: now also IC101.30 (PIO1_10-AD6-CT16B1_MAT1); no longer IC101.28 (PIO0_9-MOSI-CT16B_MAT1-SWO)
- net MOTION_DET: now also IC101.24 (PIO2_9); no longer IC101.12 (PIO2_8)
- net RED_DIM: now also IC101.29 (SWCLK-PIO0_10-SCK-CT16B0_MAT2); no longer IC101.30 (PIO1_10-AD6-CT16B1_MAT1)
- net RELAY_EN: now also IC101.45 (PIO1_5-nRTS-CT32B0_CAP0); no longer IC101.21 (PIO2_5)
- net SW1: now also P103.4; no longer P103.8
- net SW4: now also P103.2; no longer P103.10
- net WW2_DIM: now also IC101.28 (PIO0_9-MOSI-CT16B_MAT1-SWO); no longer IC101.40 (PIO1_4-AD5-CT32B1_MAT3-WAKEUP)
- net WW_DIM: now also IC101.27 (PIO0_8-MISO-CT16B0_MAT0); no longer IC101.29 (SWCLK-PIO0_10-SCK-CT16B0_MAT2)
- net RELAY_PWR_GND: now reaches P102.1 (P1), Q101.D
- net SER_USB_D: now reaches J101.3 (D+), U103.15 (USBD+)
- net ~SER_USB_D: now reaches J101.2 (D-), U103.16 (USBD-)
- net ~SER_RST: now reaches R106.1, U103.19 (RESET)
- net SER_RX_LED: now reaches D106.2 (K), U103.22 (CBUS1)
- net SER_TX_LED: now reaches D105.2 (K), U103.23 (CBUS0)
- net SER_TX_LED_R: now reaches D105.1 (A), R108.1
- net SER_RX_LED_R: now reaches D106.1 (A), R109.1
- net XB_RSSI: now reaches D102.1 (A), U102.6 (PWM/RSSI)
- net XB_RSSI_D: now reaches D102.2 (K), R101.2
- net UC_VBUS: now reaches D103.1 (A), IC101.14 (PIO0_3-USB_VBUS), J102.1 (VBUS), R104.1
- net UC_VBUS: now also C2.1
- net IIC_SCL: now reaches IC101.15 (PIO0_4-SCL)
- net IIC_SCL: now also P1.2 (P2), R2.2
- net IIC_SDA: now reaches IC101.16 (PIO0_5-SDA)
- net IIC_SDA: now also P1.3 (P3), R1.2
- net ~UC_D: now reaches IC101.19 (USB_DM), J102.2 (D-)
- net UC_D: now reaches IC101.20 (USB_DP), J102.3 (D+), R103.1
- net UC_USB_CONNECT: now reaches IC101.22 (PIO0_6-nUSB_CONNECT-SCK), Q102.G, R107.1
- net EXTRA_AD: now reaches IC101.42 (PIO1_11-AD7)
- net EXTRA_AD: now also K1.2 (PM)
- net UC_XI: now reaches C125.2, IC101.6 (XTALIN), X101.2
- net UC_XO: now reaches C124.2, IC101.7 (XTALOUT), X101.1
- net UC_D_PU: now reaches Q102.D, R103.2, R105.1
- net BOOTSEL_RESET: now reaches D108.2 (K), D109.2 (K), SW102.2
- new net USBTOUC_BOOT_SEL: D2.2 (K), U103.3 (RTS)
- new net XB_BOOT_SEL: D1.2 (K), U102.16 (/RTS/AD6/Dio6)
Other:
- note added: "Mounting Holes"
- moved on the sheet: C101, C109, C110, C111, C112, C113, C114, C123, C124, C125, C150, C151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
