File: test_Board/LPC1343_Test_Board.sch (KiCad schematic (older format))
At the start: 79 parts, among them IC101 LPC1343, J101 CONN_USB_MINI_B, J102 CONN_USB_MINI_B, P1 CONN_JST_PH_4, P2 CONN_JST_PH_3, Q102 MOSFET_P, SW1 SW_PB_MJTP1230, SW101 SW_PB_MJTP1230, SW102 SW_PB_MJTP1230, SW2 SW_PB_MJTP1230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

Commit message: Updated test board
Parts:
- removed D5: RGB_LED, symbol RGB_LED
- removed IC101: LPC1343, symbol LPC1343
- removed R103, R4: R, symbol R
- removed R104: RES_4P7K_1P_1V8W_0805, symbol RES_4P7K_1P_1V8W_0805
- removed U101: VREG_1117, symbol VREG_1117
- removed U102: XBEE, symbol XBEE
- added D5: LED_RGB_PLCC6, symbol LED_RGB_PLCC6
- added R103: RES_1P5K_1P_1V8W_0805, symbol RES_1P5K_1P_1V8W_0805
- added R104: RES_100K_1P_1V8W_0805, symbol RES_100K_1P_1V8W_0805
- added R4: RES_330_1P_1V8W_0805, symbol RES_330_1P_1V8W_0805
- added U1000: IC_LPC1343_LQFP48, symbol IC_LPC1343_LQFP48
- added U1020: IC_XBEE_SMD, symbol IC_XBEE_SMD
- added U1050: IC_MCP1700T33_SOT23, symbol IC_MCP1700T33_SOT23
- gave numbers to parts that had none: 1
- renumbered U103 to U1010
Connections:
- net labels removed: XB_RSSI_D
- wire segments 174 -> 171
Other:
- note added: "Add Series R on UC_VBUS to prevent accidental 5V short through UC"
- note added: "SW102 = Reset+Bootloader\nSW101= Reset\n"
- moved on the sheet: HW100, HW101, HW102, HW103, P1, P2, Q102

Commit message: Starting to layout the test board better.
Components have been ordered so I am working on cleaning up the layout.
Parts:
- removed D6, D7: WHITE, symbol LED
- added D6, D7: LED_GREEN_DIFF_0805, symbol LED_GREEN_DIFF_0805
Changed lines of the file:
@@
-EESchema Schematic File Version 2  date Thu 11 Oct 2012 02:05:13 PM CDT
+EESchema Schematic File Version 2  date Tue 09 Oct 2012 10:52:12 PM CDT
 LIBS:power
 LIBS:device
@@
 Sheet 1 1
 Title ""
-Date "11 oct 2012"
+Date "10 oct 2012"
 Rev ""
 Comp ""
@@
 $EndComp
 $Comp
-L LED D6
-U 1 1 50743CD0
-P 12000 2250
-F 0 "D6" H 12000 2350 50  0000 C CNN
-F 1 "WHITE" H 12000 2150 50  0000 C CNN
-	1    12000 2250
-	0    1    1    0
-$EndComp
-$Comp
-L LED D7
-U 1 1 50743CDD
-P 12450 2250
-F 0 "D7" H 12450 2350 50  0000 C CNN
-F 1 "WHITE" H 12450 2150 50  0000 C CNN
-	1    12450 2250
-	0    1    1    0
-$EndComp
-$Comp
 L GND #PWR052
 U 1 1 50743CEF
@@
 	1    0    0    -1
 $EndComp
+$Comp
+L LED_GREEN_DIFF_0805 D6
+U 1 1 5074FD7B
+P 12000 2250
+F 0 "D6" H 12000 2350 50  0000 C CNN
+F 1 "LED_GREEN_DIFF_0805" H 12000 2450 50  0001 C CNN
+F 4 "475-1410-1-ND" H 11650 2500 61  0001 L BNN "PN"
+F 5 "Green_diff" H 11800 2100 39  0000 L BNN "Val"
+F 6 "0805" H 11800 2150 39  0000 L BNN "Package"
+	1    12000 2250
+	0    1    1    0
+$EndComp
+$Comp
+L LED_GREEN_DIFF_0805 D7
+U 1 1 5074FDA1
+P 12450 2250
+F 0 "D7" H 12450 2350 50  0000 C CNN
+F 1 "LED_GREEN_DIFF_0805" H 12450 2450 50  0001 C CNN
+F 4 "475-1410-1-ND" H 12100 2500 61  0001 L BNN "PN"
+F 5 "Green_diff" H 12250 2100 39  0000 L BNN "Val"
+F 6 "0805" H 12250 2150 39  0000 L BNN "Package"
+	1    12450 2250
+	0    1    1    0
+$EndComp
 $EndSCHEMATC

Commit message: More layout
Parts:
- added C1234, C1235: CAP_0P1UF_10P_50V_X7R_0805, symbol CAP_0P1UF_10P_50V_X7R_0805
- added C12345: CAP_22UF_20P_10V_X5R_1206, symbol CAP_22UF_20P_10V_X5R_1206
Connections:
- wire segments 171 -> 172
