File: main_Board/main_Board.sch (KiCad schematic (older format))
At the start: 130 parts, among them J101 CONN_USB_MINI_B, J102 CONN_USB_MINI_B, P1 CONN_JST_PH_4, P101 CONN_JST_PH_3, P102 CONN_JST_PH_2, P103 CONN_2, P104 CONN_5X2, P105 CONN_TE_IDC_SMT_2_18GA, P106 CONN_TE_IDC_SMT_2_18GA, P107 CONN_TE_IDC_SMT_4_18GA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

Commit message: main_Board
More updates
Parts:
- added C1002, C1003, C1008, C1009, C1010, C1011: CAP_2P2UF_10P_50V_X5R_1206, symbol CAP_2P2UF_10P_50V_X5R_1206
- added C1004, C1005: CAP_1UF_10P_50V_X5R_0805, symbol CAP_1UF_10P_50V_X5R_0805
- added C1006, C1007: CAP_0P1UF_10P_50V_X7R_0805, symbol CAP_0P1UF_10P_50V_X7R_0805

Commit message: Updates to main board
Updated main board to include the analog connector.
Upadted to have a better 24V cutout plane
Parts:
- P103: Name (none) -> HEADER R/A 0p165in; PN (none) -> A30614-ND
- P104: Name (none) -> CONN_5X2; PN (none) -> 609-1767-ND
- Q102: Name (none) -> MOSFET_P_2.7A; PN (none) -> DMP2215LDICT-ND
- U1010: PN (none) -> 768-1007-1-ND
Changed lines of the file:
@@
-EESchema Schematic File Version 2  date Fri 26 Oct 2012 05:29:55 PM CDT
+EESchema Schematic File Version 2  date Tue 30 Oct 2012 11:30:43 AM CDT
 LIBS:power
 LIBS:device
@@
 Sheet 1 1
 Title ""
-Date "26 oct 2012"
+Date "30 oct 2012"
 Rev ""
 Comp ""
@@
 F 0 "Q102" H 3300 14890 60  0000 R CNN
 F 1 "MOSFET_P" H 3300 14520 60  0000 R CNN
+F 4 "DMP2215LDICT-ND" H 3300 14700 60  0001 C CNN "PN"
+F 5 "MOSFET_P_2.7A" H 3300 14700 60  0001 C CNN "Name"
 	1    3300 14700
 	-1   0    0    1
@@
 $EndComp
 $Comp
-L IC_FT232RL_SSOP28 U1010
-U 1 1 50761233
-P 6400 8400
-F 0 "U1010" H 5800 7400 60  0000 L BNN
-F 1 "IC_FT232RL_SSOP28" H 6400 7400 60  0001 L BNN
-F 3 "768-1007-1-ND" H 6400 9450 60  0001 L BNN
-F 4 "FT232RL" H 5800 9450 60  0000 L BNN "Name"
-	1    6400 8400
-	1    0    0    -1
-$EndComp
-$Comp
 L GND #PWR052
 U 1 1 50761270
@@
 F 0 "P104" H 10500 3300 60  0000 C CNN
 F 1 "CONN_5X2" V 10500 3000 50  0000 C CNN
+F 4 "609-1767-ND" H 10500 3000 60  0001 C CNN "PN"
+F 5 "CONN_5X2" H 10500 3000 60  0001 C CNN "Name"
 	1    10500 3000
 	1    0    0    -1
@@
 F 0 "P103" V 900 1500 40  0000 C CNN
 F 1 "CONN_2" V 1000 1500 40  0000 C CNN
+F 4 "A30614-ND" V 950 1500 60  0001 C CNN "PN"
+F 5 "HEADER R/A 0p165in" V 950 1500 60  0001 C CNN "Name"
 	1    950  1500
 	-1   0    0    1
@@
 	1    0    0    -1
 $EndComp
+$Comp
+L IC_FT232RL_SSOP28 U1010
+U 1 1 5090185F
+P 6400 8400
+F 0 "U1010" H 5800 7400 60  0000 L BNN
+F 1 "IC_FT232RL_SSOP28" H 6400 7400 60  0001 L BNN
+F 4 "768-1007-1-ND" H 6000 7600 60  0001 C CNN "PN"
+F 5 "FT232RL" H 6000 7600 60  0000 C CNN "Name"
+	1    6400 8400
+	1    0    0    -1
+$EndComp
