File: double_in_cab_breakout/double_in_cab_breakout.sch (KiCad schematic (older format))
At the start: 16 parts, among them P10 CONN_JST_PH_2, P11 CONN_JST_PH_2, P13 CONN_JST_PH_2, P14 CONN_JST_PH_2, P16 CONN_JST_PH_2, P17 CONN_JST_PH_2, P3 CONN_2, P4 CONN_2, Q10 MOS_N_SI2308BDS

Commit message: double_in_cab_breakout: Updated
Parts:
- removed D10: DIODE_ZENER_9P1V, symbol DIODE_ZENER_9P1V
- removed Q10: MOS_N_SI2308BDS, symbol MOS_N_SI2308BDS
- removed R10: RES_100K_1P_1V8W_0805, symbol RES_100K_1P_1V8W_0805
- removed R11: RES_0_0P_1V4_1206, symbol RES_0_0P_1V4_1206
Connections:
- net labels added: STRIP1_12V, STRIP2_12V, STRIP_GND
- net labels removed: LED_STRIP_12V, LED_STRIP_GND, SW
- wire segments 22 -> 25
Other:
- note removed: "Install R11 for high power NC switch. \nInstall R10,D10,Q10 for low power NO switch."
- moved on the sheet: P10, P11, P13, P14, P16, P17

Commit message: Updated double_in_cab_breakout
Changed to use the correct width connector.
Changed to use the terminal block.
Reduced size.
Added _panel.
Parts:
- removed C103, C104: CAP_0P1UF_10P_50V_X7R_0805, symbol CAP_0P1UF_10P_50V_X7R_0805
- removed P3, P4: CONN_2, symbol CONN_2
- added P100, P101: CONN_TERM_BLOCK_2POS_3P5MM, symbol CONN_TERM_BLOCK_2POS_3P5MM
Changed lines of the file:
@@
-EESchema Schematic File Version 2  date Wed 24 Oct 2012 09:39:02 PM CDT
+EESchema Schematic File Version 2  date Wed 31 Oct 2012 08:56:02 PM CDT
 LIBS:power
 LIBS:device
@@
 Sheet 1 1
 Title "In Cabinet LED Breakout"
-Date "25 oct 2012"
+Date "1 nov 2012"
 Rev ""
 Comp ""
@@
 $EndDescr
 $Comp
-L GND #PWR01
-U 1 1 5068AAC0
-P 4100 3650
-F 0 "#PWR01" H 4100 3650 30  0001 C CNN
-F 1 "GND" H 4100 3580 30  0001 C CNN
-	1    4100 3650
-	1    0    0    -1
-$EndComp
-$Comp
-L GND #PWR02
-U 1 1 5068AAC6
-P 3500 3650
-F 0 "#PWR02" H 3500 3650 30  0001 C CNN
-F 1 "GND" H 3500 3580 30  0001 C CNN
-	1    3500 3650
-	1    0    0    -1
-$EndComp
-$Comp
 L GND #PWR03
 U 1 1 5068AACC
@@
 F 1 "+24V" H 2900 3350 30  0000 C CNN
 	1    2900 3250
-	1    0    0    -1
-$EndComp
-$Comp
-L +24V #PWR07
-U 1 1 5068AAEE
-P 3500 3250
-F 0 "#PWR07" H 3500 3200 20  0001 C CNN
-F 1 "+24V" H 3500 3350 30  0000 C CNN
-	1    3500 3250
-	1    0    0    -1
-$EndComp
-$Comp
-L +24V #PWR08
-U 1 1 5068AAFA
-P 4100 3250
-F 0 "#PWR08" H 4100 3200 20  0001 C CNN
-F 1 "+24V" H 4100 3350 30  0000 C CNN
-	1    4100 3250
 	1    0    0    -1
 $EndComp
@@
 $EndComp
 $Comp
-L CAP_0P1UF_10P_50V_X7R_0805 C103
-U 1 1 5074DABB
-P 3500 3450
-F 0 "C103" H 3550 3550 50  0000 L CNN
-F 1 "CAP_0P1UF_10P_50V_X7R_0805" H 3600 3250 50  0001 L CNN
-F 4 "311-1140-1-ND" H 4000 3150 60  0001 C CNN "PN"
-F 5 "0.1uF" H 3375 3500 39  0000 R BNN "Val"
-F 6 "0805" H 3375 3350 39  0000 R BNN "Package"
-F 7 "10%" H 3375 3450 39  0000 R BNN "Tol"
-F 8 "50V" H 3375 3400 39  0000 R BNN "Voltage"
-	1    3500 3450
-	1    0    0    -1
-$EndComp
-$Comp
-L CAP_0P1UF_10P_50V_X7R_0805 C104
-U 1 1 5074DAEC
-P 4100 3450
-F 0 "C104" H 4150 3550 50  0000 L CNN
-F 1 "CAP_0P1UF_10P_50V_X7R_0805" H 4200 3250 50  0001 L CNN
-F 4 "311-1140-1-ND" H 4600 3150 60  0001 C CNN "PN"
-F 5 "0.1uF" H 3975 3500 39  0000 R BNN "Val"
-F 6 "0805" H 3975 3350 39  0000 R BNN "Package"
-F 7 "10%" H 3975 3450 39  0000 R BNN "Tol"
-F 8 "50V" H 3975 3400 39  0000 R BNN "Voltage"
-	1    4100 3450
-	1    0    0    -1
-$EndComp
-$Comp
 L CONN_JST_PH_2 P10
 U 1 1 5074E11A
@@
 $EndComp
 $Comp
-L CONN_2 P4
-U 1 1 508349BE
-P 6150 2400
-F 0 "P4" V 6100 2400 40  0000 C CNN
-F 1 "CONN_2" V 6200 2400 40  0000 C CNN
-	1    6150 2400
-	0    1    1    0
-$EndComp
-$Comp
-L CONN_2 P3
-U 1 1 508349CB
-P 5750 2400
-F 0 "P3" V 5700 2400 40  0000 C CNN
-F 1 "CONN_2" V 5800 2400 40  0000 C CNN
-	1    5750 2400
-	0    1    1    0
-$EndComp
-$Comp
 L GND #PWR09
 U 1 1 508349E0
@@
 Text Label 7700 4650 1    40   ~ 0
 STRIP_GND
+$Comp
+L CONN_TERM_BLOCK_2POS_3P5MM P100
+U 1 1 5091BA69
+P 5750 2400
+F 0 "P100" V 5750 2400 40  0000 C CNN
+F 1 "CONN_TERM_BLOCK_2POS_3P5MM" H 5700 2650 40  0001 C CNN
+F 4 "A98036-ND" H 5750 2100 60  0001 C CNN "PN"
+F 5 "TRM_BLK_2" H 5450 2200 40  0000 L BNN "Name"
+	1    5750 2400
+	0    1    1    0
+$EndComp
+$Comp
+L CONN_TERM_BLOCK_2POS_3P5MM P101
+U 1 1 5091BA8B
+P 6150 2400
+F 0 "P101" V 6150 2400 40  0000 C CNN
+F 1 "CONN_TERM_BLOCK_2POS_3P5MM" H 6100 2650 40  0001 C CNN
+F 4 "A98036-ND" H 6150 2100 60  0001 C CNN "PN"
+F 5 "TRM_BLK_2" H 5850 2200 40  0000 L BNN "Name"
+	1    6150 2400
+	0    1    1    0
+$EndComp
 $EndSCHEMATC
